File: Cat-Phones-DK-V1.kicad_pcb (KiCad board)
At the start: 2 copper layers, 97 x 62.4 mm, 51 parts, among them J1 USB_C, J10 GPIO-25, J11 Battery Charger IN, J12 GPIO-26, J13 DAC-Power, J14 Conn_01x04, J15 Battery VCC, J16 Battery GND, J17 DAC-Power, J18 AudioJack4, J19 Conn_01x02, J2 Conn_01x08, J3 GPIO, J4 ESP-TX, J5 ESP-RX, J6 GPIO-0, J7 EN, J8 Power-Switch, J9 GPIO-27, Q1 SS8050, Q2 SS8050, Q3 FS8205A, U1 CH340C, U2 ESP32-WROOM-32UE, U3 AP2112K-3.3TRG1, U4 TP4057, U5 PCM5102A, U6 DW01A

Commit message: 💕
Parts:
- added J15: Conn_01x04, Connector_PinSocket_2.54mm:PinSocket_1x04_P2.54mm_Vertical, F.Cu at (185.2, 77.1)
- J20: renamed from J19; footprint Connector_PinSocket_2.54mm:PinSocket_1x02_P2.54mm_Vertical -> Connector_PinSocket_2.00mm:PinSocket_1x02_P2.00mm_Vertical
- moved J18 13.9 mm to (164.5, 108.5)
- moved J11 4.84 mm to (160.9, 111.0)
- moved J16 0.74 mm to (170.8, 108.5)
- moved J17 0.73 mm to (174.3, 111.0)
- renumbered J15 to J16, J16 to J17, J17 to J18, J18 to J19
Routing:
- net VBUS: track 13.9 -> 111.2 mm, vias 0 -> 4
- net +5V: track 102.9 -> 141.3 mm
- net -BATT: track 0.00 -> 38.2 mm
- net +BATT: track 32.9 -> 66.3 mm, vias 0 -> 1
- net Net-(D1-A): track 52.3 -> 55.0 mm
- net +3V3: track 99.8 -> 98.8 mm
- net Net-(J16-Pin_1): track 4.33 -> 5.09 mm
- net Net-(J17-Pin_2): track 23.0 -> 23.8 mm
- net GND: vias 27 -> 32
- added copper zone on B.Cu, net GND
Other:
- board text added: "+"
- board text added: "-"
- board text added: "2.5v-6v"
- board text added: "5v"
- board text added: "Battery"
- board text added: "Battery IN"
- board text added: "Battery to protect"
- board text added: "Burning Area"
- board text added: "CatPhones Dev-Kit V1"
- board text added: "Discharge"
- board text added: "EN"
- board text added: "ESP32 WROOM"
- board text added: "External BMS"
- board text added: "Fuck it I do it my way area"
- board text added: "GND"
- board text added: "GPIO"
- board text added: "I love you all"
- board text added: "I2c DAC"
- board text added: "IN"
- board text added: "IN OUT"
- board text added: "IO0"
- board text added: "OUT"
- board text added: "Power"
- board text added: "Power curcid"
- board text added: "RX"
- board text added: "TX"
- board text added: "USB to serial"
- board text added: "charge"
